Commit message: point cloud octomap

File: src/motoman/motoman_hc10_support/urdf/hc10.sensor.xacro (robot description, xacro)
@@ -5,5 +5,5 @@
     <!-- Attach Kinect to tool -->
     <joint type="fixed" name="tool0_sensor">
-        <origin xyz="0.15 -1 0.1" rpy="0 0 1.57"/>
+        <origin xyz="0 0 0" rpy="1.57 -1.57 0"/>
         <child link="camera_depth_frame"/>
         <parent link="tool0"/>

File: src/motoman/motoman_hc10_support/urdf/hc10.xacro (robot description, xacro)
@@ -8,3 +8,4 @@
   <xacro:hc10_gazebo prefix=""/>
   <xacro:include filename="$(find motoman_hc10_support)/urdf/hc10.sensor.xacro"/>
+  <xacro:include filename="$(find motoman_hc10_support)/urdf/kinect_camera.gazebo.xacro"/>
 </robot>
